Commit message: chang model feature

File: Multiagent-Reaction/multiagent_reaction/resources/simplegoal.urdf (robot description, URDF)
Before this commit: robot simplegoal, 1 links, 0 joints
Links:
- link base_link: geometry collision cylinder length=0.2 radius=0.25; visual cylinder length=1 radius=1

Commit message: model fix

File: Multiagent-Reaction/multiagent_reaction/resources/simplegoal.urdf (robot description, URDF)
Before this commit: robot simplegoal, 1 links, 0 joints
Links:
- link base_link: mass 1 -> 4

File: Multiagent-Reaction/multiagent_reaction/resources/simpleplane.urdf (robot description, URDF)
Before this commit: robot simpleplane, 1 links, 0 joints
Links:
- link base_link: geometry collision box size=400 400 0.1; visual box size=400 400 0.1
